File: 4x4_keyboard_2.1.brd (EAGLE design)
At the start: 72 x 134.4 mm, 83 parts, among them U2 AMS1117-5.0

Commit message: make component placement perfect
Parts:
- moved LED3 12.3 mm to (52.6, 154.3), turned to 90 degrees
- moved R6 12.2 mm to (55.2, 154.3), turned to 270 degrees
- moved D18 1.40 mm to (51.4, 160.1)
- moved C3 1.19 mm to (51.0, 148.2)
- moved U$18 0.85 mm to (61.2, 151.4)
- moved C7 0.51 mm to (55.1, 160.0)
- moved C1 0.50 mm to (51.0, 145.8)
Routing:
- net VCC: track 96.1 -> 92.0 mm
- net N$4: track 11.3 -> 9.87 mm
- net GND: track 10.4 -> 10.9 mm, vias 104 -> 118

Commit message: remove the logo and prog led for testing
Parts:
- removed U$18: (no value), SparkFun-Aesthetics:SMART_BASIC_LOGO
- added LED2: Green, led:SML0805
- added R8: 1K, audio amplifier example:R0603
- moved R7 2.54 mm to (26.3, 159.4)
- moved S2 1.00 mm to (21.5, 159.6)
- renumbered SV2 to IN
Connections:
- new net N$16: LED2.A, R8.2
- new net PROG_LED: LED2.C
- new net PRO_LED: U$17.12
- net VCC: now also R8.1
Routing:
- net RESET: track 64.9 -> 57.6 mm, vias 0 -> 2
- net N$16: track 0.00 -> 3.08 mm
- net VCC: track 92.0 -> 93.6 mm, vias 0 -> 2
- net SCK: track 41.8 -> 41.6 mm, vias 2 -> 0
- net MISO: track 36.4 -> 36.3 mm, vias 2 -> 0
