File: eagle files/4x4_keyboard_2.1.brd (EAGLE design)
At the start: 72 x 134.4 mm, 83 parts, among them U2 AMS1117-5.0

Commit message: design files
Parts:
- removed U$18: (no value), SparkFun-Aesthetics:SMART_BASIC_LOGO
- added LED2: Green, led:SML0805
- added R8: 1K, audio amplifier example:R0603
- moved R7 2.54 mm to (26.3, 159.4)
- moved S2 1.00 mm to (21.5, 159.6)
- moved U$2 0.05 mm to (32.2, 101.5)
Connections:
- new net N$16: LED2.A, R8.2
- new net PROG_LED: LED2.C
- new net PRO_LED: U$17.12
- net VCC: now also R8.1
Routing:
- net ROW3: track 156.4 -> 177.0 mm
- net ROW4: track 172.6 -> 190.5 mm, vias 2 -> 6
- net ROW2: track 139.2 -> 154.1 mm
- net ROW1: track 119.0 -> 133.7 mm
- net RESET: track 64.9 -> 57.6 mm, vias 0 -> 2
- net N$16: track 0.00 -> 3.08 mm
- net VCC: track 92.0 -> 93.6 mm, vias 0 -> 2
- net SCK: track 41.8 -> 41.6 mm, vias 2 -> 0
- net MISO: track 36.4 -> 36.3 mm, vias 2 -> 0
Other:
- board size 72 x 134.4 mm -> 72 x 136 mm
